File: PIC18 DEV BOARD.sch (EAGLE design)
At the start: 23 parts, among them IC2 7805TV, J2 J5MM, J5 J10MM, X1 22-23-2081, X3 22-23-2021, X4 22-23-2041

Commit message: Add files via upload
Parts:
- removed J5: J10MM, jumper:J10MM
- removed R1, R2: (no value), rcl:R-US_0207/10
- removed R4: (no value), rcl:R-TRIMM64P
- removed SL2: (no value), con-amp-quick:M05S
- added D1: 1N4004, diode:1N4004
- added J1: J12MM, jumper:J12MM
- added J3: 9V DC IN, con-jack:JACK-PLUG0
- added J4: J15MM, jumper:J15MM
- added S2: P/SEL, switch:320-916
- added X10: 22-23-2021, con-molex:22-23-2021
- added X2: (no value), con-molex:22-23-2061
- added X8, X9: 22-23-2041, con-molex:22-23-2041
- X3: value 22-23-2021 -> (none); device con-molex:22-23-2021 -> con-molex:22-23-2061
- X4: value 22-23-2041 -> 22-23-2081; device con-molex:22-23-2041 -> con-molex:22-23-2081
Connections:
- removed net N$1 (its old number): U$1.CCP1/P1A/RC2, X3-2.S
- removed net N$19: C4.1, IC2.VO, JP1.2, R1.2, R2.2, R3.2, R4.A, R7.2, SL2-1.S, U$1.VDD@0, U$1.VDD@1, X1-2.S
- new net N$10: U$1.CCP2/AN9/RB3, X2-4.S
- new net N$17: J1.1, U$1.SDI/SDA/RC4
- new net N$18: J4.1, U$1.SDO/RC5
- new net N$20: U$1.TX/CK/RC6, X10-1.S
- new net N$24: U$1.RX/DT/RC7, X10-2.S
- new net N$26: U$1.PSP1/RD1, X4-2.S
- new net N$27: U$1.PSP2/RD2, X4-3.S
- new net N$29: J1.2, X3-5.S
- new net N$32: U$1.PSP4/RD4, X4-5.S
- new net N$33: U$1.P1B/PSP5/RD5, X4-6.S
- new net N$34: U$1.P1C/PSP6/RD6, X4-7.S
- new net N$37: U$1._WR/AN6/RE1, X1-7.S
- new net N$39: U$1._CS/AN7/RE2, X1-8.S
- new net N$41: U$1.VREF+/AN3/RA3, X1-4.S
- new net N$42: J4.2, X3-6.S
- new net N$43: D1.A, S2.P
- new net N$44: C3.1, D1.C, IC2.VI, X6-1.KL, X7-1.KL
- new net N$45: S2.S, X5-1.KL
- new net N$47: C4.1, IC2.VO, JP1.2, R3.2, R7.2, U$1.VDD@0, U$1.VDD@1, X9-1.S, X9-2.S, X9-3.S, X9-4.S
- new net N$9: U$1.INT2/AN8/RB2, X2-3.S
- net GND: now also J3.1, J3.2, X5-2.KL, X6-2.KL, X7-2.KL, X8-1.S, X8-2.S, X8-3.S, X8-4.S; no longer R4.E, SL2-2.S, X1-1.S, X5-1.KL, X6-1.KL, X7-1.KL
- net N$11: now also U$1.KBI0/AN11/RB4, X2-5.S; no longer J5.1, U$1.INT0/FLT0/AN12/RB0
- net N$12: now also U$1.KBI1/PGM/RB5, X2-6.S; no longer U$1.I1OSI/CCP2/RC1, X3-1.S
- net N$13: now also U$1.T1OSO/T13CKI/RC0, X3-1.S; no longer U$1.VREF-/CVREF/AN2/RA2, X4-1.S
- net N$14: now also U$1.I1OSI/CCP2/RC1, X3-2.S; no longer U$1.VREF+/AN3/RA3, X4-2.S
- net N$15: now also U$1.CCP1/P1A/RC2, X3-3.S; no longer U$1.T0CKI/C1OUT/RA4, X4-3.S
- net N$16: now also U$1.SCK/SCL/RC3, X3-4.S; no longer U$1._SS/HLVDIN/C2OUT/AN4/RA5, X4-4.S
- net N$2: now also U$1.AN0/RA0, X1-1.S; no longer U$1.P1D/PSP7/RD7, X1-3.S
- net N$25: now also U$1.PSP0/RD0, X4-1.S; no longer R4.S, U$1.AN0/RA0
- net N$28: now also U$1.PSP3/RD3, X4-4.S; no longer C3.1, IC2.VI, X5-2.KL, X6-2.KL, X7-2.KL
- net N$3: now also U$1.AN1/RA1, X1-2.S; no longer U$1.P1C/PSP6/RD6, X1-4.S
- net N$35: now also U$1.P1D/PSP7/RD7, X4-8.S; no longer R1.1, SL2-4.S, U$1.SCK/SCL/RC3
- net N$36: now also U$1._RD/AN5/RE0, X1-6.S; no longer R2.1, SL2-3.S, U$1.SDI/SDA/RC4
- net N$4: now also U$1.VREF-/CVREF/AN2/RA2, X1-3.S; no longer U$1.P1B/PSP5/RD5, X1-5.S
- net N$5: now also J3.3, S2.O; no longer U$1.PSP4/RD4, X1-6.S
- net N$6: now also U$1._SS/HLVDIN/C2OUT/AN4/RA5, X1-5.S; no longer U$1.PSP3/RD3, X1-7.S
- net N$7: now also U$1.INT0/FLT0/AN12/RB0, X2-1.S; no longer U$1.PSP2/RD2, X1-8.S
- net N$8: now also U$1.INT1/AN10/RB1, X2-2.S; no longer J5.2, SL2-5.S
Other:
- moved on the sheet: X1-1, X1-2, X1-3, X1-4, X1-5, X1-6, X1-7, X1-8, X3-1, X3-2, X4-1, X4-2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
